File: Hbrige_MotorController/Hbrige_MotorController.kicad_pcb (KiCad board)
At the start: 2 copper layers, 82.5 x 61.2 mm, 66 parts, among them J1 Conn_01x05_Female, J2 Conn_01x04_Female, J3 Conn_01x04_Female, J4 Conn_02x03_Odd_Even, J5 Screw_Terminal_01x02, M1 Motor_DC, Q1 IRF3205, Q2 IRF3205, Q3 IRF3205, Q4 IRF3205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

Commit message: Add files via upload
Parts:
- C5, C6, C7, C8: value 22pf -> 18pf
- J1: value Conn_01x05_Female -> Conn_01x05_Male
- J2, J3: value Conn_01x04_Female -> Conn_01x04_Male
- R12: value k5 -> 1k
- R5, R6, R7, R8: value 27k -> 220
- U1: value ATmega328P-A -> ATmega328PB-A
- moved C2 65.7 mm to (150.1, 88.0)
- moved ? 65.7 mm to (168.8, 133.2)
- moved ? 65.7 mm to (94.3, 133.2)
- moved ? 65.7 mm to (94.3, 80.0)
- moved ? 65.7 mm to (168.8, 80.0)
- moved C1 65.7 mm to (158.1, 111.0)
- moved C10 65.7 mm to (113.8, 94.0)
- moved C11 65.7 mm to (106.8, 123.0)
- moved C12 65.7 mm to (97.8, 123.0)
- moved C13 65.7 mm to (96.3, 106.5)
- moved C14 65.7 mm to (104.3, 117.0)
- moved C15 65.7 mm to (128.6, 106.8)
- moved C17 65.7 mm to (115.1, 106.8)
- moved C18 65.7 mm to (147.3, 106.8)
- moved C19 65.7 mm to (139.3, 96.8)
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Connections:
- U1 pad 19: A6 -> unconnected-(U1-Pad19)
- U1 pad 22: A7 -> unconnected-(U1-Pad22)
- U1 pad 3: GND -> unconnected-(U1-Pad3)
Routing:
- net GND: track 18.8 -> 14.2 mm, vias 10 -> 12
