File: Hbrige_MotorController/drivers.kicad_sch (KiCad schematic)
At the start: 31 parts, among them M1 Motor_DC, Q1 IRF3205, Q2 IRF3205, Q3 IRF3205, Q4 IRF3205, U4 IRS2104, U5 IRS2104

Commit message: Add files via upload
Parts:
- R12: value k5 -> 1k
- R5, R6, R7, R8: value 27k -> 220
Changed lines of the file:
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@@
       (effects (font (size 1.27 1.27)) (justify right))
     )
-    (property "Value" "k5" (id 1) (at 104.14 85.0899 0)
+    (property "Value" "1k" (id 1) (at 104.14 85.0899 0)
       (effects (font (size 1.27 1.27)) (justify right))
     )
@@
     (in_bom yes) (on_board yes) (fields_autoplaced)
     (property "Reference" "R6" (id 0) (at 92.71 101.6 90))
-    (property "Value" "27k" (id 1) (at 92.71 104.14 90))
+    (property "Value" "220" (id 1) (at 92.71 104.14 90))
     (property "Footprint" "Resistor_SMD:R_0603_1608Metric_Pad0.98x0.95mm_HandSolder" (id 2) (at 92.71 109.728 90)
       (effects (font (size 1.27 1.27)) hide)
@@
     (in_bom yes) (on_board yes)
     (property "Reference" "R7" (id 0) (at 179.07 102.87 90))
-    (property "Value" "27k" (id 1) (at 179.07 100.33 90))
+    (property "Value" "220" (id 1) (at 179.07 100.33 90))
     (property "Footprint" "Resistor_SMD:R_0603_1608Metric_Pad0.98x0.95mm_HandSolder" (id 2) (at 179.07 96.012 90)
       (effects (font (size 1.27 1.27)) hide)
@@
     (in_bom yes) (on_board yes) (fields_autoplaced)
     (property "Reference" "R8" (id 0) (at 179.07 68.58 90))
-    (property "Value" "27k" (id 1) (at 179.07 71.12 90))
+    (property "Value" "220" (id 1) (at 179.07 71.12 90))
     (property "Footprint" "Resistor_SMD:R_0603_1608Metric_Pad0.98x0.95mm_HandSolder" (id 2) (at 179.07 73.152 90)
       (effects (font (size 1.27 1.27)) hide)
@@
     (in_bom yes) (on_board yes) (fields_autoplaced)
     (property "Reference" "R5" (id 0) (at 92.71 78.74 90))
-    (property "Value" "27k" (id 1) (at 92.71 81.28 90))
+    (property "Value" "220" (id 1) (at 92.71 81.28 90))
     (property "Footprint" "Resistor_SMD:R_0603_1608Metric_Pad0.98x0.95mm_HandSolder" (id 2) (at 92.71 86.868 90)
       (effects (font (size 1.27 1.27)) hide)
