File: Hbrige_MotorController/untitled.kicad_sch (KiCad schematic)
At the start: 31 parts, among them J1 Conn_01x05_Female, J2 Conn_01x04_Female, J3 Conn_01x04_Female, J4 Conn_02x03_Odd_Even, J5 Screw_Terminal_01x02, U1 ATmega328P-A, U2 MCP2515-xSO, U3 MCP2551-I-SN, Y1 8MHz, Y2 16MHz

Commit message: Add files via upload
Parts:
- removed U1: ATmega328P-A, Package_QFP:TQFP-32_7x7mm_P0.8mm, symbol MCU_Microchip_ATmega:ATmega328P-A
- added U1: ATmega328PB-A, Package_QFP:TQFP-32_7x7mm_P0.8mm, symbol MCU_Microchip_ATmega:ATmega328PB-A
- C5, C6, C7, C8: value 22pf -> 26pf
- J1: value Conn_01x05_Female -> Conn_01x05_Male
- J2, J3: value Conn_01x04_Female -> Conn_01x04_Male
Connections:
- net +5V: now also U1.18 (AVCC), U1.4 (VCC), U1.6 (PE1)
- net A0: now also U1.23 (PC0)
- net A1: now also U1.24 (PC1)
- net A2: now also U1.25 (PC2)
- net A3: now also U1.26 (PC3)
- net CS: now also U1.14 (PB2)
- net D6: now also U1.10 (PD6)
- net D8: now also U1.12 (PB0)
- net EN: now also U1.11 (PD7)
- net GND: now also U1.21 (GND), U1.5 (GND)
- net INT1: now also U1.32 (PD2)
- net INT2: now also U1.1 (PD3)
- net INT_CAN: now also U1.2 (PD4)
- net MISO: now also U1.16 (PB4)
- net MOSI: now also U1.15 (PB3)
- net PWM1: now also U1.9 (PD5)
- net PWM2: now also U1.13 (PB1)
- net RST: now also U1.29 (~{RESET}/PC6)
- net SCK: now also U1.17 (PB5)
- net SCL: now also U1.28 (PC5)
- net SDA: now also U1.27 (PC4)
- net at C5.2, Y2.1: now also U1.7 (XTAL1/PB6)
- net at C6.2, Y2.2: now also U1.8 (XTAL2/PB7)
- net at R3.2: now also U1.31 (PD1)
- net at C4.2: now also U1.20 (AREF)
- net at R2.2: now also U1.30 (PD0)
- no-connect marks 7 -> 10
Other:
- note added: "CL = (26pf * 26pf)/(26pf * 26pf) + 5 = 18pf"
